File: connectors.sch (KiCad schematic (older format))
At the start: 3 parts, among them P501 USB_OTG, X501 CON_SWD, X502 SUB-D9

Commit message: Add Fit, Manufacturer, MPN fields
Parts:
- P501: Fit (none) -> fit:; MPN (none) -> 47491-0001; Manufacturer (none) -> Molex
- X501: Fit (none) -> fit: none
- X502: Fit (none) -> fit:; MPN (none) -> 156-1209T-E; Manufacturer (none) -> Kobiconn
Changed lines of the file:
@@
 F 2 "Connect:DB9M_CI" H 7900 3150 60  0001 C CNN
 F 3 "" H 7900 3150 60  0000 C CNN
+F 4 "fit: " H 7950 3150 50  0001 C CNN "Fit"
+F 5 "156-1209T-E" H 7950 3150 50  0001 C CNN "MPN"
+F 6 "Kobiconn" H 7950 3150 50  0001 C CNN "Manufacturer"
 	1    7950 3150
 	1    0    0    -1
@@
 AR Path="/56F635D5" Ref="X501"  Part="1"
 AR Path="/56F568C1/56F635D5" Ref="X501"  Part="1"
-F 0 "X501" H 6050 3600 60  0000 C CNN
-F 1 "CON_SWD" H 6050 2800 60  0000 C CNN
+F 0 "X501" H 6228 3279 60  0000 L CNN
+F 1 "CON_SWD" H 6228 3173 60  0000 L CNN
 F 2 "tagconnect:TC2030-NL" H 6000 3200 60  0001 C CNN
 F 3 "" H 6000 3200 60  0000 C CNN
+F 4 "fit: none" H 6228 3094 25  0000 L CNN "Fit"
 	1    6050 3200
 	1    0    0    -1
@@
 F 2 "usb:Molex-Micro-USB-B-Middle-Mount" V 4250 3000 50  0001 C CNN
 F 3 "" V 4250 3000 50  0000 C CNN
+F 4 "fit: " H 4300 3100 50  0001 C CNN "Fit"
+F 5 "47491-0001" H 4300 3100 50  0001 C CNN "MPN"
+F 6 "Molex" H 4300 3100 50  0001 C CNN "Manufacturer"
 	1    4300 3100
 	0    1    1    0
