File: leds.sch (KiCad schematic (older format))
At the start: 6 parts

Commit message: Add Fit, Manufacturer, MPN fields
Parts:
- D601: Fit (none) -> fit:; MPN (none) -> APT1608SGC; Manufacturer (none) -> Kingbright
- D602: Fit (none) -> fit:; MPN (none) -> APT1608YC; Manufacturer (none) -> Kingbright
- D603: Fit (none) -> fit:; MPN (none) -> APT1608EC; Manufacturer (none) -> Kingbright
- R601, R602, R603: Fit (none) -> fit:
Changed lines of the file:
@@
 F 2 "LEDs:LED_0603" H 5900 3650 50  0001 C CNN
 F 3 "" H 5900 3650 50  0000 C CNN
+F 4 "fit: " H 5900 3650 50  0001 C CNN "Fit"
+F 5 "APT1608SGC" H 5900 3650 50  0001 C CNN "MPN"
+F 6 "Kingbright" H 5900 3650 50  0001 C CNN "Manufacturer"
 	1    5900 3650
 	-1   0    0    1
@@
 F 2 "LEDs:LED_0603" H 5900 4000 50  0001 C CNN
 F 3 "" H 5900 4000 50  0000 C CNN
+F 4 "fit: " H 5900 4000 50  0001 C CNN "Fit"
+F 5 "APT1608YC" H 5900 4000 50  0001 C CNN "MPN"
+F 6 "Kingbright" H 5900 4000 50  0001 C CNN "Manufacturer"
 	1    5900 4000
 	-1   0    0    1
@@
 F 2 "LEDs:LED_0603" H 5900 4350 50  0001 C CNN
 F 3 "" H 5900 4350 50  0000 C CNN
+F 4 "fit: " H 5900 4350 50  0001 C CNN "Fit"
+F 5 "APT1608EC" H 5900 4350 50  0001 C CNN "MPN"
+F 6 "Kingbright" H 5900 4350 50  0001 C CNN "Manufacturer"
 	1    5900 4350
 	-1   0    0    1
@@
 F 2 "Resistors_SMD:R_0603" V 5380 3650 50  0001 C CNN
 F 3 "" H 5450 3650 50  0000 C CNN
+F 4 "fit: " H 5450 3650 50  0001 C CNN "Fit"
 	1    5450 3650
 	0    1    1    0
@@
 F 2 "Resistors_SMD:R_0603" V 5380 4000 50  0001 C CNN
 F 3 "" H 5450 4000 50  0000 C CNN
+F 4 "fit: " H 5450 4000 50  0001 C CNN "Fit"
 	1    5450 4000
 	0    1    1    0
@@
 F 2 "Resistors_SMD:R_0603" V 5380 4350 50  0001 C CNN
 F 3 "" H 5450 4350 50  0000 C CNN
+F 4 "fit: " H 5450 4350 50  0001 C CNN "Fit"
 	1    5450 4350
 	0    1    1    0

Commit message: Update Silkscreen and add netnames
Changed lines of the file:
@@
 $EndComp
 Wire Wire Line
-	5150 3550 5150 4350
+	5150 3550 5150 3650
 Connection ~ 5150 3650
 Connection ~ 5150 4000
@@
 Wire Wire Line
 	5600 4350 5700 4350
+Wire Wire Line
+	5150 3650 5150 4000
+Wire Wire Line
+	5150 4000 5150 4350
 $EndSCHEMATC
