File: CAN.sch (KiCad schematic (older format))
At the start: 5 parts, among them U401 TJA1051/3

Commit message: Add Fit, Manufacturer, MPN fields
Parts:
- C402, C403, R401: Fit (none) -> fit:
- R402: Fit (none) -> fit: none
- U401: Fit (none) -> fit:; MPN (none) -> TJA1051T/3/1J; Manufacturer (none) -> NXP
Changed lines of the file:
@@
 F 2 "Housings_SOIC:SOIC-8_3.9x4.9mm_Pitch1.27mm" H 5750 3750 60  0001 C CNN
 F 3 "" H 5750 3750 60  0000 C CNN
+F 4 "TJA1051T/3/1J" H 5750 3600 50  0001 C CNN "MPN"
+F 5 "NXP" H 5750 3600 50  0001 C CNN "Manufacturer"
+F 6 "fit: " H 5750 3600 50  0001 C CNN "Fit"
 	1    5750 3600
 	1    0    0    -1
@@
 F 2 "Capacitors_SMD:C_0603" H 6000 4650 50  0001 C CNN
 F 3 "" H 6000 4650 50  0000 C CNN
+F 4 "fit: " H 6000 4650 50  0001 C CNN "Fit"
 	1    6000 4650
 	1    0    0    -1
@@
 F 2 "Capacitors_SMD:C_0603" H 5700 4650 50  0001 C CNN
 F 3 "" H 5700 4650 50  0000 C CNN
+F 4 "fit: " H 5700 4650 50  0001 C CNN "Fit"
 	1    5700 4650
 	1    0    0    -1
@@
 F 2 "Resistors_SMD:R_0603" V 4480 3100 50  0001 C CNN
 F 3 "" H 4550 3100 50  0000 C CNN
+F 4 "fit: " H 4550 3100 50  0001 C CNN "Fit"
 	1    4550 3100
 	1    0    0    -1
@@
 F 3 "" H 4550 2950 50  0000 C CNN
 	1    4550 2950
-	1    0    0    -1
-$EndComp
-$Comp
-L candleLight-rescue:R R402
-U 1 1 56F69E23
-P 6650 3150
-F 0 "R402" V 6730 3150 50  0000 C CNN
-F 1 "dnp" V 6650 3150 50  0000 C CNN
-F 2 "Resistors_SMD:R_0805" V 6580 3150 50  0001 C CNN
-F 3 "" H 6650 3150 50  0000 C CNN
-	1    6650 3150
 	1    0    0    -1
 $EndComp
@@
 Wire Wire Line
 	6650 3000 6950 3000
+$Comp
+L candleLight-rescue:R R402
+U 1 1 56F69E23
+P 6650 3150
+F 0 "R402" V 6730 3150 50  0000 C CNN
+F 1 "dnp" V 6650 3150 50  0000 C CNN
+F 2 "Resistors_SMD:R_0805" V 6580 3150 50  0001 C CNN
+F 3 "" H 6650 3150 50  0000 C CNN
+F 4 "fit: none" V 6775 3150 25  0000 C CNN "Fit"
+	1    6650 3150
+	1    0    0    -1
+$EndComp
 $EndSCHEMATC

Commit message: Add Cap voltage rating, Put PCB ref on cupper, add note for variants
Parts:
- C402, C403: CapRatedVoltage (none) -> 10V
Changed lines of the file:
@@
 F 3 "" H 6000 4650 50  0000 C CNN
 F 4 "fit: " H 6000 4650 50  0001 C CNN "Fit"
+F 5 "10V" H 6125 4650 25  0000 C CNN "CapRatedVoltage"
 	1    6000 4650
 	1    0    0    -1
@@
 F 3 "" H 5700 4650 50  0000 C CNN
 F 4 "fit: " H 5700 4650 50  0001 C CNN "Fit"
+F 5 "10V" H 5825 4650 25  0000 C CNN "CapRatedVoltage"
 	1    5700 4650
 	1    0    0    -1
