File: candleLight.sch (KiCad schematic (older format))
At the start: 3 parts

Commit message: Add Fit, Manufacturer, MPN fields
Parts:
- FID101, FID102, FID103: Fit (none) -> fit:
Changed lines of the file:
@@
 F 2 "Fiducials:Fiducial_1mm_Dia_2.54mm_Outer_CopperTop" H 9900 950 50  0001 C CNN
 F 3 "" H 9900 950 50  0000 C CNN
+F 4 "fit: " H 9900 950 50  0001 C CNN "Fit"
 	1    9900 950
 	1    0    0    -1
@@
 F 2 "Fiducials:Fiducial_1mm_Dia_2.54mm_Outer_CopperTop" H 9900 1350 50  0001 C CNN
 F 3 "" H 9900 1350 50  0000 C CNN
+F 4 "fit: " H 9900 1350 50  0001 C CNN "Fit"
 	1    9900 1350
 	1    0    0    -1
@@
 F 2 "Fiducials:Fiducial_1mm_Dia_2.54mm_Outer_CopperTop" H 9900 1750 50  0001 C CNN
 F 3 "" H 9900 1750 50  0000 C CNN
+F 4 "fit: " H 9900 1750 50  0001 C CNN "Fit"
 	1    9900 1750
 	1    0    0    -1

Commit message: Add Cap voltage rating, Put PCB ref on cupper, add note for variants
Other:
- note added: "Variants:\n=======\nV1: Complete assembly\nV2: V1 but without THT-components (SMD only) [Created manually in Post]\nV3: V1 but only THT-components (no SMD) [Created manually in Post]\n"
Changed lines of the file:
@@
 Comp "Linux Automation GmbH"
 Comment1 "released"
-Comment2 "candleLight-S01-R01-V01-C00"
+Comment2 "candleLight-S01-R01-V01"
 Comment3 "github.com/linux-automation/candlelight-S01"
 Comment4 ""
@@
 	1    0    0    -1
 $EndComp
+Text Notes 750  6975 0    60   ~ 0
+Variants:\n=======\nV1: Complete assembly\nV2: V1 but without THT-components (SMD only) [Created manually in Post]\nV3: V1 but only THT-components (no SMD) [Created manually in Post]\n
 $EndSCHEMATC

Commit message: Add linux automation logo
Parts:
- added NB101: LAG_logo, logo:lag_rocket_10mmx10.4mm, symbol logo:LAG_logo
Changed lines of the file:
@@
 Text Notes 750  6975 0    60   ~ 0
 Variants:\n=======\nV1: Complete assembly\nV2: V1 but without THT-components (SMD only) [Created manually in Post]\nV3: V1 but only THT-components (no SMD) [Created manually in Post]\n
+$Comp
+L logo:LAG_logo NB101
+U 1 1 6040F88F
+P 9825 2100
+F 0 "NB101" H 9903 2153 60  0000 L CNN
+F 1 "LAG_logo" H 9903 2047 60  0000 L CNN
+F 2 "logo:lag_rocket_10mmx10.4mm" H 9825 2100 60  0001 C CNN
+F 3 "" H 9825 2100 60  0001 C CNN
+	1    9825 2100
+	1    0    0    -1
+$EndComp
 $EndSCHEMATC
